Commit message: tb3p_description: read sensor extrinsics from calibration.yaml

File: tb3p_description/urdf/tb3p_burger.urdf.xacro (robot description, xacro)
@@ -7,4 +7,17 @@
 -->
 <robot name="tb3p_burger" xmlns:xacro="http://ros.org/wiki/xacro">
+  <!-- ===== 캘리브레이션 파일 읽기 ===== -->
+  <xacro:arg name="calib_file" default="$(find tb3p_description)/config/calibration.yaml"/>
+  <xacro:property name="calib" value="${xacro.load_yaml('$(arg calib_file)')}"/>
+  <!-- 센서 조인트: 위치와 방향을 calibration.yaml에서 읽는다 -->
+  <xacro:macro name="calibrated_joint" params="joint key">
+    <xacro:property name="s" value="${calib['sensors'][key]}"/>
+    <joint name="${joint}" type="fixed">
+      <parent link="${s['parent']}"/>
+      <child link="${s['child']}"/>
+      <origin xyz="${s['xyz'][0]} ${s['xyz'][1]} ${s['xyz'][2]}"
+              rpy="${s['rpy'][0]} ${s['rpy'][1]} ${s['rpy'][2]}"/>
+    </joint>
+  </xacro:macro>
   <!-- ===== 색 ===== -->
   <material name="light_black"><color rgba="0.4 0.4 0.4 1.0"/></material>
@@ -94,9 +107,5 @@
   </gazebo>
   <!-- ===== IMU (OpenCR) ===== -->
-  <joint name="imu_joint" type="fixed">
-    <parent link="base_link"/>
-    <child link="imu_link"/>
-    <origin xyz="-0.032 0 0.068" rpy="0 0 0"/>
-  </joint>
+  <xacro:calibrated_joint joint="imu_joint" key="imu"/>
   <link name="imu_link"/>
   <gazebo reference="imu_link">
@@ -121,9 +130,5 @@
   </gazebo>
   <!-- ===== 2D LiDAR (현재 LDS-01 사양 그대로, 세션 4에서 LDS-02로 교체) ===== -->
-  <joint name="scan_joint" type="fixed">
-    <parent link="base_link"/>
-    <child link="base_scan"/>
-    <origin xyz="-0.032 0 0.172" rpy="0 0 0"/>
-  </joint>
+  <xacro:calibrated_joint joint="scan_joint" key="lidar"/>
   <link name="base_scan">
     <visual>

Commit message: Sensor specs from datasheets: LDS-03 LiDAR, IMU noise densities in YAML (ICM-20648, BMI055), depth noise

File: tb3p_description/urdf/tb3p_burger.urdf.xacro (robot description, xacro)
@@ -2,14 +2,18 @@
 <!--
   tb3p Burger 설계도 (단일 원본)
-  - 위치(조인트 origin): turtlebot3_description의 URDF 값 = 공칭값
+  - 센서 위치: calib_file(YAML)의 sensors, 나머지 위치: turtlebot3_description URDF 값
   - 물리 값(질량, 관성, 마찰): turtlebot3_gazebo의 model.sdf 값 (Gazebo에서 검증된 값)
   - Gazebo 센서는 링크 기준점에 놓음(센서 pose 없음) → Gazebo 위치 = TF 위치
+  - 센서 사양: LiDAR LDS-03, 몸체 IMU ICM-20648 (데이터시트, 2026-10-10 확인)
+  - IMU 노이즈: calib_file의 imu_noise (노이즈 밀도) → σ = 밀도 × √rate
+  - 스위치: calib_file, sim, truth (+ tb3p_camera_sim.urdf.xacro의 enable_infra)
 -->
 <robot name="tb3p_burger" xmlns:xacro="http://ros.org/wiki/xacro">
-  <!-- ===== 캘리브레이션 파일 읽기 ===== -->
+  <!-- ===== 스위치와 캘리브레이션 파일 ===== -->
   <xacro:arg name="calib_file" default="$(find tb3p_description)/config/calibration.yaml"/>
   <xacro:arg name="sim" default="false"/>
+  <xacro:arg name="truth" default="false"/>
   <xacro:property name="calib" value="${xacro.load_yaml('$(arg calib_file)')}"/>
-  <!-- 센서 조인트: 위치와 방향을 calibration.yaml에서 읽는다 -->
+  <!-- 센서 조인트: 위치와 방향을 YAML의 sensors에서 읽는다 -->
   <xacro:macro name="calibrated_joint" params="joint key">
     <xacro:property name="s" value="${calib['sensors'][key]}"/>
@@ -20,4 +24,23 @@
               rpy="${s['rpy'][0]} ${s['rpy'][1]} ${s['rpy'][2]}"/>
     </joint>
+  </xacro:macro>
+  <!-- Gazebo IMU 주기와 노이즈: YAML의 imu_noise에서 읽어 샘플당 σ로 환산 -->
+  <xacro:macro name="gz_imu_noise" params="key">
+    <xacro:property name="n" value="${calib['imu_noise'][key]}"/>
+    <xacro:property name="sg" value="${n['gyro_noise_density'] * n['rate'] ** 0.5}"/>
+    <xacro:property name="sa" value="${n['accel_noise_density'] * n['rate'] ** 0.5}"/>
+    <update_rate>${n['rate']}</update_rate>
+    <imu>
+      <angular_velocity>
+        <x><noise type="gaussian"><mean>0.0</mean><stddev>${sg}</stddev></noise></x>
+        <y><noise type="gaussian"><mean>0.0</mean><stddev>${sg}</stddev></noise></y>
+        <z><noise type="gaussian"><mean>0.0</mean><stddev>${sg}</stddev></noise></z>
+      </angular_velocity>
+      <linear_acceleration>
+        <x><noise type="gaussian"><mean>0.0</mean><stddev>${sa}</stddev></noise></x>
+        <y><noise type="gaussian"><mean>0.0</mean><stddev>${sa}</stddev></noise></y>
+        <z><noise type="gaussian"><mean>0.0</mean><stddev>${sa}</stddev></noise></z>
+      </linear_acceleration>
+    </imu>
   </xacro:macro>
   <!-- ===== 색 ===== -->
@@ -87,4 +110,5 @@
   <xacro:wheel side="right" y="-0.08" mesh="right_tire.stl"/>
   <!-- ===== 뒤쪽 캐스터 (URDF는 볼 조인트가 없어 고정 + 마찰 0으로 미끄러지게) ===== -->
+  <!-- 바퀴 바닥보다 1 mm 높음 → Gazebo 로봇이 약 0.7° 앞들림 (W7 IMU 정렬 시험 재료로 유지) -->
   <joint name="caster_back_joint" type="fixed">
     <parent link="base_link"/>
@@ -107,5 +131,5 @@
     <mu2>0.0</mu2>
   </gazebo>
-  <!-- ===== IMU (OpenCR) ===== -->
+  <!-- ===== 몸체 IMU (OpenCR ICM-20648) ===== -->
   <xacro:calibrated_joint joint="imu_joint" key="imu"/>
   <link name="imu_link"/>
@@ -113,22 +137,11 @@
     <sensor name="tb3_imu" type="imu">
       <always_on>true</always_on>
-      <update_rate>200</update_rate>
       <topic>imu</topic>
       <gz_frame_id>imu_link</gz_frame_id>
-      <imu>
-        <angular_velocity>
-          <x><noise type="gaussian"><mean>0.0</mean><stddev>2e-4</stddev></noise></x>
-          <y><noise type="gaussian"><mean>0.0</mean><stddev>2e-4</stddev></noise></y>
-          <z><noise type="gaussian"><mean>0.0</mean><stddev>2e-4</stddev></noise></z>
-        </angular_velocity>
-        <linear_acceleration>
-          <x><noise type="gaussian"><mean>0.0</mean><stddev>1.7e-2</stddev></noise></x>
-          <y><noise type="gaussian"><mean>0.0</mean><stddev>1.7e-2</stddev></noise></y>
-          <z><noise type="gaussian"><mean>0.0</mean><stddev>1.7e-2</stddev></noise></z>
-        </linear_acceleration>
-      </imu>
+      <xacro:gz_imu_noise key="base_imu"/>
     </sensor>
   </gazebo>
-  <!-- ===== 2D LiDAR (현재 LDS-01 사양 그대로, 세션 4에서 LDS-02로 교체) ===== -->
+  <!-- ===== 2D LiDAR (LDS-03: 0.05–12 m, 10 Hz, 0.9° = 400점, 정확도 ±10/±20 mm) ===== -->
+  <!-- 모양과 판 위 높이는 아직 LDS-01 기준 (LDS-03 치수 확인 후 교체) -->
   <xacro:calibrated_joint joint="scan_joint" key="lidar"/>
   <link name="base_scan">
@@ -151,8 +164,8 @@
   </link>
   <gazebo reference="base_scan">
-    <sensor name="hls_lfcd_lds" type="gpu_lidar">
+    <sensor name="lds_03" type="gpu_lidar">
       <always_on>true</always_on>
       <visualize>true</visualize>
-      <update_rate>5</update_rate>
+      <update_rate>10</update_rate>
       <topic>scan</topic>
       <gz_frame_id>base_scan</gz_frame_id>
@@ -160,15 +173,17 @@
         <scan>
           <horizontal>
-            <samples>360</samples>
+            <!-- 400점, 0.9° 간격: 마지막 점이 첫 점과 겹치지 않게 2π × 399/400 까지 -->
+            <samples>400</samples>
             <resolution>1.0</resolution>
             <min_angle>0.0</min_angle>
-            <max_angle>6.28</max_angle>
+            <max_angle>${2 * pi * 399 / 400}</max_angle>
           </horizontal>
         </scan>
         <range>
-          <min>0.12</min>
-          <max>3.5</max>
-          <resolution>0.015</resolution>
+          <min>0.05</min>
+          <max>12.0</max>
+          <resolution>0.001</resolution>
         </range>
+        <!-- 정확도 ±20 mm(1 m 이상)를 약 2σ로 보고 σ = 10 mm (Gazebo는 거리와 무관한 상수 σ만 지원) -->
         <noise>
           <type>gaussian</type>
@@ -181,4 +196,5 @@
   <!-- ===== 추가 층: Jetson과 새 판 ===== -->
   <xacro:include filename="$(find tb3p_description)/urdf/tb3p_mast.urdf.xacro"/>
+  <!-- ===== D435i 카메라 ===== -->
   <xacro:include filename="$(find tb3p_description)/urdf/tb3p_camera.urdf.xacro"/>
   <!-- ===== Gazebo 플러그인: 바퀴 구동과 바퀴 각도 보고 ===== -->

File: tb3p_description/urdf/tb3p_camera.urdf.xacro (robot description, xacro)
@@ -8,4 +8,7 @@
   - (나) 상자 안 렌즈 배치: sim:=true일 때만 설계도가 만든다 (use_nominal_extrinsics)
         실제 로봇에서는 realsense 드라이버가 공장 캘리브레이션 값으로 발행
+  - truth:=true (Gazebo 정답 모델 전용): 나사를 지나는 수직축 둘레로 도는 마운트 관절.
+        /sim/camera_mount_yaw_cmd (rad)로 실행 중에 각도를 바꿔 드리프트를 흉내 낸다.
+        공칭 모델(/tf)에는 이 관절이 없으므로 로봇은 카메라가 돌아간 것을 모른다.
   - 브래킷: 기존 맨 위판 위 3 mm 판, 앞 지지대 사이로 판 끝 밖까지 (모양만, 추정 치수)
   - 이 파일은 tb3p_mast.urdf.xacro 다음에 include해야 함 (plate_top_z, plate_grey 사용)
@@ -14,11 +17,58 @@
   <xacro:include filename="$(find realsense2_description)/urdf/_d435i.urdf.xacro"/>
   <xacro:property name="cam" value="${calib['sensors']['camera']}"/>
+  <xacro:property name="cam_xyz" value="${cam['xyz'][0]} ${cam['xyz'][1]} ${cam['xyz'][2]}"/>
+  <xacro:property name="cam_rpy" value="${cam['rpy'][0]} ${cam['rpy'][1]} ${cam['rpy'][2]}"/>
   <xacro:property name="bracket_thk" value="0.003"/>
-  <!-- ===== D435i: 위치는 YAML, 내부 좌표계는 sim 스위치 ===== -->
-  <xacro:sensor_d435i parent="${cam['parent']}" name="camera"
-                      use_nominal_extrinsics="$(arg sim)">
-    <origin xyz="${cam['xyz'][0]} ${cam['xyz'][1]} ${cam['xyz'][2]}"
-            rpy="${cam['rpy'][0]} ${cam['rpy'][1]} ${cam['rpy'][2]}"/>
-  </xacro:sensor_d435i>
+  <!-- ===== 공칭·실제 로봇: 카메라는 고정 ===== -->
+  <xacro:unless value="$(arg truth)">
+    <xacro:sensor_d435i parent="${cam['parent']}" name="camera"
+                        use_nominal_extrinsics="$(arg sim)">
+      <origin xyz="${cam_xyz}" rpy="${cam_rpy}"/>
+    </xacro:sensor_d435i>
+  </xacro:unless>
+  <!-- ===== 정답 모델(Gazebo): 나사 축 둘레로 도는 마운트 관절 ===== -->
+  <xacro:if value="$(arg truth)">
+    <joint name="camera_mount_yaw_joint" type="revolute">
+      <parent link="${cam['parent']}"/>
+      <child link="camera_mount_link"/>
+      <origin xyz="${cam_xyz}" rpy="0 0 0"/>
+      <axis xyz="0 0 1"/>
+      <limit lower="-0.2" upper="0.2" effort="10.0" velocity="1.0"/>
+    </joint>
+    <link name="camera_mount_link">
+      <inertial>
+        <origin xyz="0 0 0"/>
+        <mass value="0.005"/>
+        <inertia ixx="1e-06" ixy="0" ixz="0" iyy="1e-06" iyz="0" izz="1e-06"/>
+      </inertial>
+    </link>
+    <!-- 관절 각도 0이면 고정일 때와 같은 자리: 위치는 관절에, 방향은 여기에 -->
+    <xacro:sensor_d435i parent="camera_mount_link" name="camera"
+                        use_nominal_extrinsics="$(arg sim)">
+      <origin xyz="0 0 0" rpy="${cam_rpy}"/>
+    </xacro:sensor_d435i>
+    <gazebo>
+      <!-- 목표 각도(rad)를 받아 관절을 그 각도로 돌려 유지 -->
+      <plugin filename="gz-sim-joint-position-controller-system"
+              name="gz::sim::systems::JointPositionController">
+        <joint_name>camera_mount_yaw_joint</joint_name>
+        <topic>sim/camera_mount_yaw_cmd</topic>
+        <use_velocity_commands>true</use_velocity_commands>
+        <p_gain>5.0</p_gain>
+        <i_gain>0.0</i_gain>
+        <d_gain>0.0</d_gain>
+        <cmd_max>0.5</cmd_max>
+        <cmd_min>-0.5</cmd_min>
+      </plugin>
+      <!-- 정답 TF용 관절 각도 보고 (/truth/joint_states) -->
+      <plugin filename="gz-sim-joint-state-publisher-system"
+              name="gz::sim::systems::JointStatePublisher">
+        <topic>truth/joint_states</topic>
+        <joint_name>camera_mount_yaw_joint</joint_name>
+        <joint_name>wheel_left_joint</joint_name>
+        <joint_name>wheel_right_joint</joint_name>
+      </plugin>
+    </gazebo>
+  </xacro:if>
   <!-- ===== 브래킷 (모양만): x 0.020 ~ 0.064, 폭 36 mm (앞 지지대 y=±24 사이) ===== -->
   <joint name="camera_bracket_joint" type="fixed">

File: tb3p_description/urdf/tb3p_camera_sim.urdf.xacro (robot description, xacro)
@@ -5,15 +5,17 @@
   - 카메라는 일반 좌표계(x 앞)에 붙이고, 메시지 frame_id는 optical 좌표계(z 앞)로
   - IMU는 합친 형태(unite_imu_method)로 /camera/camera/imu, frame camera_imu_optical_frame
+    노이즈는 YAML imu_noise.camera_imu (BMI055 데이터시트)
   - 해상도 848x480 @ 30 Hz, 시야각: RGB 69°, 깊이·IR 87° (D435i 데이터시트)
+  - 깊이 노이즈: 실제는 거리 제곱에 비례 (2 m에서 2% 이내), Gazebo는 상수 σ만 지원 → σ 10 mm
   - IR 카메라 두 개는 enable_infra:=true일 때만 (렌더링 부하 때문에 기본 끔)
   - 점구름은 Gazebo가 아니라 depth_image_proc로 만든다 (Gazebo 점구름은 일반 좌표계 방향)
-  - 노이즈, 측정 거리: 세션 4에서 데이터시트 값으로 조정
 -->
 <robot xmlns:xacro="http://ros.org/wiki/xacro">
   <xacro:arg name="enable_infra" default="false"/>
   <xacro:if value="$(arg sim)">
-    <!-- 카메라 센서 하나 -->
+    <!-- 카메라 센서 하나 (noise_stddev 0이면 노이즈 없음) -->
     <xacro:macro name="gz_camera"
-                 params="link frame name type image_topic info_topic hfov format near far">
+                 params="link frame name type image_topic info_topic hfov format near far
+                         noise_stddev:=0.0">
       <gazebo reference="${link}">
         <sensor name="${name}" type="${type}">
@@ -35,4 +37,11 @@
               <far>${far}</far>
             </clip>
+            <xacro:if value="${noise_stddev > 0}">
+              <noise>
+                <type>gaussian</type>
+                <mean>0.0</mean>
+                <stddev>${noise_stddev}</stddev>
+              </noise>
+            </xacro:if>
           </camera>
         </sensor>
@@ -51,5 +60,6 @@
                      name="d435i_depth" type="depth_camera"
                      image_topic="${ns}/depth/image_rect_raw" info_topic="${ns}/depth/camera_info"
-                     hfov="${fov_depth}" format="R_FLOAT32" near="0.2" far="10.0"/>
+                     hfov="${fov_depth}" format="R_FLOAT32" near="0.2" far="10.0"
+                     noise_stddev="0.01"/>
     <!-- IR 왼쪽, 오른쪽 (흑백): 필요할 때만 -->
     <xacro:if value="$(arg enable_infra)">
@@ -75,7 +85,7 @@
       <sensor name="d435i_imu" type="imu">
         <always_on>true</always_on>
-        <update_rate>200</update_rate>
         <topic>${ns}/imu</topic>
         <gz_frame_id>camera_imu_optical_frame</gz_frame_id>
+        <xacro:gz_imu_noise key="camera_imu"/>
       </sensor>
     </gazebo>

Commit message: Session 10: IMU noise sweep with repeated trials
- imu_noise_scale arg in xacro and calib_rig launch (headless gui:=false)
- sweep_imu_noise.sh: record, convert, Kalibr imu-cam, score per scale
- repeat_sweep.sh: N trials per scale, stale-process and IMU-noise checks
- plot_sweep_trials.py: per-trial dots, median line, CSV
- results: translation median 0.68/1.09/4.02/6.88 mm at x1/x3/x10/x30

File: tb3p_description/urdf/tb3p_burger.urdf.xacro (robot description, xacro)
@@ -10,38 +10,6 @@
 -->
 <robot name="tb3p_burger" xmlns:xacro="http://ros.org/wiki/xacro">
-  <!-- ===== 스위치와 캘리브레이션 파일 ===== -->
-  <xacro:arg name="calib_file" default="$(find tb3p_description)/config/calibration.yaml"/>
-  <xacro:arg name="sim" default="false"/>
-  <xacro:arg name="truth" default="false"/>
-  <xacro:property name="calib" value="${xacro.load_yaml('$(arg calib_file)')}"/>
-  <!-- 센서 조인트: 위치와 방향을 YAML의 sensors에서 읽는다 -->
-  <xacro:macro name="calibrated_joint" params="joint key">
-    <xacro:property name="s" value="${calib['sensors'][key]}"/>
-    <joint name="${joint}" type="fixed">
-      <parent link="${s['parent']}"/>
-      <child link="${s['child']}"/>
-      <origin xyz="${s['xyz'][0]} ${s['xyz'][1]} ${s['xyz'][2]}"
-              rpy="${s['rpy'][0]} ${s['rpy'][1]} ${s['rpy'][2]}"/>
-    </joint>
-  </xacro:macro>
-  <!-- Gazebo IMU 주기와 노이즈: YAML의 imu_noise에서 읽어 샘플당 σ로 환산 -->
-  <xacro:macro name="gz_imu_noise" params="key">
-    <xacro:property name="n" value="${calib['imu_noise'][key]}"/>
-    <xacro:property name="sg" value="${n['gyro_noise_density'] * n['rate'] ** 0.5}"/>
-    <xacro:property name="sa" value="${n['accel_noise_density'] * n['rate'] ** 0.5}"/>
-    <update_rate>${n['rate']}</update_rate>
-    <imu>
-      <angular_velocity>
-        <x><noise type="gaussian"><mean>0.0</mean><stddev>${sg}</stddev></noise></x>
-        <y><noise type="gaussian"><mean>0.0</mean><stddev>${sg}</stddev></noise></y>
-        <z><noise type="gaussian"><mean>0.0</mean><stddev>${sg}</stddev></noise></z>
-      </angular_velocity>
-      <linear_acceleration>
-        <x><noise type="gaussian"><mean>0.0</mean><stddev>${sa}</stddev></noise></x>
-        <y><noise type="gaussian"><mean>0.0</mean><stddev>${sa}</stddev></noise></y>
-        <z><noise type="gaussian"><mean>0.0</mean><stddev>${sa}</stddev></noise></z>
-      </linear_acceleration>
-    </imu>
-  </xacro:macro>
+  <!-- ===== 스위치, 캘리브레이션 파일, 공통 매크로 (tb3p_common) ===== -->
+  <xacro:include filename="$(find tb3p_description)/urdf/tb3p_common.urdf.xacro"/>
   <!-- ===== 색 ===== -->
   <material name="light_black"><color rgba="0.4 0.4 0.4 1.0"/></material>

Commit message: Session 15: wheel errors in sim truth, UMBmark driving and wheel calibration

File: tb3p_description/urdf/tb3p_burger.urdf.xacro (robot description, xacro)
@@ -8,4 +8,6 @@
   - IMU 노이즈: calib_file의 imu_noise (노이즈 밀도) → σ = 밀도 × √rate
   - 스위치: calib_file, sim, truth (+ tb3p_camera_sim.urdf.xacro의 enable_infra)
+  - 바퀴: 모양(반지름, 좌우 위치)은 calib_file의 wheels, Gazebo DiffDrive의 계산 값은 늘 공칭
+    (config/calibration.yaml) → 정답 모델에서는 "실제 바퀴"와 "로봇이 믿는 바퀴"가 다르다 (W7)
 -->
 <robot name="tb3p_burger" xmlns:xacro="http://ros.org/wiki/xacro">
@@ -41,9 +43,12 @@
   </link>
   <!-- ===== 바퀴 (매크로: 좌우를 한 번에 정의) ===== -->
-  <xacro:macro name="wheel" params="side y mesh">
+  <!-- 반지름과 간격은 calib_file의 wheels. 바퀴 중심 높이 = 반지름 (base_link는 바닥 위 10 mm) -->
+  <xacro:property name="wheels" value="${calib['wheels']}"/>
+  <xacro:macro name="wheel" params="side sign mesh">
+    <xacro:property name="r" value="${wheels['radius_' + side]}"/>
     <joint name="wheel_${side}_joint" type="continuous">
       <parent link="base_link"/>
       <child link="wheel_${side}_link"/>
-      <origin xyz="0 ${y} 0.023" rpy="-1.57 0 0"/>
+      <origin xyz="0 ${sign * wheels['separation'] / 2} ${r - 0.010}" rpy="-1.57 0 0"/>
       <axis xyz="0 0 1"/>
     </joint>
@@ -58,5 +63,5 @@
       <collision>
         <origin xyz="0 0 0" rpy="0 0 0"/>
-        <geometry><cylinder length="0.018" radius="0.033"/></geometry>
+        <geometry><cylinder length="0.018" radius="${r}"/></geometry>
       </collision>
       <inertial>
@@ -75,6 +80,6 @@
     </gazebo>
   </xacro:macro>
-  <xacro:wheel side="left"  y="0.08"  mesh="left_tire.stl"/>
-  <xacro:wheel side="right" y="-0.08" mesh="right_tire.stl"/>
+  <xacro:wheel side="left"  sign="1"  mesh="left_tire.stl"/>
+  <xacro:wheel side="right" sign="-1" mesh="right_tire.stl"/>
   <!-- ===== 뒤쪽 캐스터 (URDF는 볼 조인트가 없어 고정 + 마찰 0으로 미끄러지게) ===== -->
   <!-- 바퀴 바닥보다 1 mm 높음 → Gazebo 로봇이 약 0.7° 앞들림 (W7 IMU 정렬 시험 재료로 유지) -->
@@ -168,10 +173,13 @@
   <xacro:include filename="$(find tb3p_description)/urdf/tb3p_truth.urdf.xacro"/>
   <!-- ===== Gazebo 플러그인: 바퀴 구동과 바퀴 각도 보고 ===== -->
+  <!-- DiffDrive는 로봇 펌웨어 역할: 명령 -> 바퀴 속도, 바퀴 각도 -> /odom 을 늘 공칭 바퀴 값으로 계산 -->
+  <xacro:property name="nominal_wheels"
+                  value="${xacro.load_yaml('$(find tb3p_description)/config/calibration.yaml')['wheels']}"/>
   <gazebo>
     <plugin filename="gz-sim-diff-drive-system" name="gz::sim::systems::DiffDrive">
       <left_joint>wheel_left_joint</left_joint>
       <right_joint>wheel_right_joint</right_joint>
-      <wheel_separation>0.160</wheel_separation>
-      <wheel_radius>0.033</wheel_radius>
+      <wheel_separation>${nominal_wheels['separation']}</wheel_separation>
+      <wheel_radius>${(nominal_wheels['radius_left'] + nominal_wheels['radius_right']) / 2}</wheel_radius>
       <max_linear_acceleration>1.0</max_linear_acceleration>
       <topic>cmd_vel</topic>

Commit message: Session 16: IMU mount angles (gravity + steady arcs), lever arm, sphere wheel collision

File: tb3p_description/urdf/tb3p_burger.urdf.xacro (robot description, xacro)
@@ -44,4 +44,9 @@
   <!-- ===== 바퀴 (매크로: 좌우를 한 번에 정의) ===== -->
   <!-- 반지름과 간격은 calib_file의 wheels. 바퀴 중심 높이 = 반지름 (base_link는 바닥 위 10 mm) -->
+  <!-- 바퀴 충돌 모양 (세션 16): 공식 모델의 원통(폭 18 mm) 대신 같은 반지름의 구.
+       원통일 때 Gazebo 로봇이 바퀴 사이 가운데가 아니라 오른쪽 약 9 mm(= 폭의 절반) 점을
+       중심으로 돌았다 (정답 위치로 확인). 원통-바닥 접촉이 원통 한쪽 끝 한 점으로 계산되는
+       것으로 보이며, 축 회전을 -1.57에서 정확한 π/2로 바꿔도 그대로였다.
+       구는 접촉점이 늘 바퀴 중심 바로 아래라서 회전 중심이 가운데가 된다 -->
   <xacro:property name="wheels" value="${calib['wheels']}"/>
   <xacro:macro name="wheel" params="side sign mesh">
@@ -50,10 +55,10 @@
       <parent link="base_link"/>
       <child link="wheel_${side}_link"/>
-      <origin xyz="0 ${sign * wheels['separation'] / 2} ${r - 0.010}" rpy="-1.57 0 0"/>
+      <origin xyz="0 ${sign * wheels['separation'] / 2} ${r - 0.010}" rpy="${-pi / 2} 0 0"/>
       <axis xyz="0 0 1"/>
     </joint>
     <link name="wheel_${side}_link">
       <visual>
-        <origin xyz="0 0 0" rpy="1.57 0 0"/>
+        <origin xyz="0 0 0" rpy="${pi / 2} 0 0"/>
         <geometry>
           <mesh filename="package://turtlebot3_description/meshes/wheels/${mesh}" scale="0.001 0.001 0.001"/>
@@ -63,5 +68,5 @@
       <collision>
         <origin xyz="0 0 0" rpy="0 0 0"/>
-        <geometry><cylinder length="0.018" radius="${r}"/></geometry>
+        <geometry><sphere radius="${r}"/></geometry>
       </collision>
       <inertial>
